Commit message: v4.8 -control ros2 onprogress

File: src/arduinobot_description/urdf/arduinobot.urdf.xacro (robot description, xacro)
@@ -1,4 +1,6 @@
 <?xml version="1.0"?>
 <robot xmlns:xacro="http://www.ros.org/wiki/xacro" name="arduinobot">
+    <xacro:include filename="$(find arduinobot_description)/urdf/arduinobot_gazebo.xacro"/>
+    <xacro:include filename="$(find arduinobot_description)/urdf/arduinobot_ros2_control.xacro"/>
     <xacro:property name="PI"  value="3.14159"/>
     <xacro:property name="effort"  value="30"/>
@@ -13,4 +15,17 @@
         </inertial>
     </xacro:macro>
+    <xacro:macro name="default_transmission" params="number">
+        <transmission name="transmission_${number}">
+            <plugin>
+                transmission_interface/SimpleTransmission
+            </plugin>
+            <actuator name="motor_${number}" role="actuator1"/>
+            <joint name="joint_${number}" role="joint1">
+                <mechanical_reduction>
+                    1.0
+                </mechanical_reduction>
+            </joint>
+        </transmission>
+    </xacro:macro>
     <link name="world"/>
     <link name="base_link">
@@ -165,4 +180,8 @@
         <limit lower="0.0" upper="${PI/2}" effort="${effort}" velocity="${velocity}"/>
     </joint>
+    <xacro:default_transmission number="1"/>
+    <xacro:default_transmission number="2"/>
+    <xacro:default_transmission number="3"/>
+    <xacro:default_transmission number="4"/>
     <link name="camera_link">
         <xacro:default_inertial mass="0.001"/>
